File: MRCS-Remote-Switch-Motor-Controller.brd (EAGLE design)
At the start: 38 x 38 mm, 13 parts, among them CON1 CONNECTOR-M03350-LOCK, J1 J1, J2 J2, M1 WIREPAD2,54/1,1, M8 WIREPAD2,54/1,1, Q1 2N3904, U1 TC4428A

Commit message: Added work files to gitignore and label changes
Added work files to gitignore and made labels on board 56 mil rather than 32 so they can be read more easily
Parts:
- added U$1: (no value), MRCSLogoBtm:MRCSLOGOBTM
- added U$2: (no value), MRCS-prop65warningBtm:CA-PROP65WARNING
- R4, R5: value 1500 -> 1.5K
- R6: value 1000 -> 1K
Other:
- board text added: "RSMC V1.9"
Changed lines of the file:
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@@
 <layer number="23" name="tOrigins" color="15" fill="1" visible="yes" active="yes"/>
 <layer number="24" name="bOrigins" color="15" fill="1" visible="no" active="yes"/>
-<layer number="25" name="tNames" color="7" fill="1" visible="no" active="yes"/>
+<layer number="25" name="tNames" color="7" fill="1" visible="yes" active="yes"/>
 <layer number="26" name="bNames" color="7" fill="1" visible="no" active="yes"/>
 <layer number="27" name="tValues" color="7" fill="1" visible="yes" active="yes"/>
@@
 <layer number="50" name="dxf" color="7" fill="1" visible="no" active="no"/>
 <layer number="51" name="tDocu" color="7" fill="1" visible="yes" active="yes"/>
-<layer number="52" name="bDocu" color="7" fill="1" visible="no" active="yes"/>
+<layer number="52" name="bDocu" color="7" fill="1" visible="yes" active="yes"/>
 <layer number="53" name="tGND_GNDA" color="7" fill="9" visible="no" active="no"/>
 <layer number="54" name="bGND_GNDA" color="1" fill="9" visible="no" active="no"/>
@@
 <layer number="99" name="Anatomie" color="7" fill="1" visible="no" active="no"/>
 <layer number="125" name="_tNames" color="14" fill="1" visible="yes" active="yes"/>
-<layer number="127" name="_tValues" color="14" fill="1" visible="yes" active="yes"/>
 </layers>
 <board>
@@
 <text x="8.89" y="34.29" size="1.016" layer="21" font="vector" ratio="10" rot="R90">M+</text>
 <text x="33.02" y="34.29" size="1.016" layer="21" font="vector" ratio="10" rot="R90">M-</text>
+<text x="36.83" y="26.035" size="1.778" layer="52" font="vector" ratio="10" rot="MR270">RSMC V1.9</text>
 <text x="18.415" y="6.985" size="0.8128" layer="125" font="vector">C1</text>
 <text x="8.4725" y="1.76499375" size="0.8128" layer="125" font="vector" rot="R180">CON1</text>
@@
 <text x="1.27" y="36.449" size="0.8128" layer="125" font="vector" ratio="10">M1</text>
 <text x="35.56" y="36.449" size="0.8128" layer="125" font="vector" ratio="10">M8</text>
-<text x="36.195" y="7.62" size="0.8128" layer="125" font="vector" ratio="10" rot="R270">Q1</text>
-<text x="23.495" y="18.415" size="0.8128" layer="125" font="vector" ratio="10" rot="R270">R3</text>
-<text x="28.575" y="18.415" size="0.8128" layer="125" font="vector" ratio="10" rot="R270">R4</text>
-<text x="31.115" y="18.415" size="0.8128" layer="125" font="vector" ratio="10" rot="R270">R5</text>
-<text x="26.035" y="18.415" size="0.8128" layer="125" font="vector" ratio="10" rot="R270">R6</text>
+<text x="36.195" y="7.62" size="1.27" layer="125" font="vector" ratio="10" rot="R270">Q1</text>
+<text x="23.495" y="18.415" size="1.6764" layer="125" font="vector" ratio="10" rot="R270">R3</text>
+<text x="28.575" y="18.415" size="1.6764" layer="125" font="vector" ratio="10" rot="R270">R4</text>
+<text x="31.115" y="18.415" size="1.6764" layer="125" font="vector" ratio="10" rot="R270">R5</text>
+<text x="26.035" y="18.415" size="1.6764" layer="125" font="vector" ratio="10" rot="R270">R6</text>
 <text x="13.97" y="5.588" size="1.27" layer="125" font="vector">ST1</text>
 <text x="12.954" y="19.304" size="0.8128" layer="125" font="vector" ratio="10">U1</text>
@@
 </element>
 <element name="Q1" library="SPCoast" package="TO-92-MS013" value="2N3904" x="33.02" y="6.35" smashed="yes" rot="R270">
-<attribute name="NAME" x="36.195" y="7.62" size="0.8128" layer="25" ratio="10" rot="R270"/>
+<attribute name="NAME" x="36.195" y="7.62" size="1.27" layer="25" ratio="10" rot="R270"/>
 <attribute name="VALUE" x="29.845" y="8.89" size="1.016" layer="27" ratio="10" rot="R270"/>
 </element>
 <element name="R3" library="SPCoast" package="AXIAL-0.4-RES" value="1M" x="24.13" y="19.05" smashed="yes" rot="R270">
-<attribute name="NAME" x="23.495" y="18.415" size="0.8128" layer="25" font="vector" ratio="10" rot="R270"/>
-<attribute name="VALUE" x="23.749" y="21.336" size="0.8128" layer="21" font="vector" ratio="10" rot="R270"/>
-</element>
-<element name="R4" library="SPCoast" package="AXIAL-0.4-RES" value="1500" x="29.21" y="19.05" smashed="yes" rot="R270">
-<attribute name="NAME" x="28.575" y="18.415" size="0.8128" layer="25" font="vector" ratio="10" rot="R270"/>
-<attribute name="VALUE" x="28.829" y="21.336" size="0.8128" layer="21" font="vector" ratio="10" rot="R270"/>
-</element>
-<element name="R5" library="SPCoast" package="AXIAL-0.4-RES" value="1500" x="31.75" y="19.05" smashed="yes" rot="R270">
-<attribute name="NAME" x="31.115" y="18.415" size="0.8128" layer="25" font="vector" ratio="10" rot="R270"/>
-<attribute name="VALUE" x="31.369" y="21.336" size="0.8128" layer="21" font="vector" ratio="10" rot="R270"/>
-</element>
-<element name="R6" library="SPCoast" package="AXIAL-0.4-RES" value="1000" x="26.67" y="19.05" smashed="yes" rot="R270">
-<attribute name="NAME" x="26.035" y="18.415" size="0.8128" layer="25" font="vector" ratio="10" rot="R270"/>
-<attribute name="VALUE" x="26.289" y="21.336" size="0.8128" layer="21" font="vector" ratio="10" rot="R270"/>
+<attribute name="NAME" x="23.495" y="18.415" size="1.6764" layer="25" font="vector" ratio="10" rot="R270"/>
+<attribute name="VALUE" x="23.114" y="21.971" size="1.6764" layer="21" font="vector" ratio="10" rot="R270"/>
+</element>
+<element name="R4" library="SPCoast" package="AXIAL-0.4-RES" value="1.5K" x="29.21" y="19.05" smashed="yes" rot="R270">
+<attribute name="NAME" x="28.575" y="18.415" size="1.6764" layer="25" font="vector" ratio="10" rot="R270"/>
+<attribute name="VALUE" x="28.194" y="22.606" size="1.4224" layer="21" font="vector" ratio="10" rot="R270"/>
+</element>
+<element name="R5" library="SPCoast" package="AXIAL-0.4-RES" value="1.5K" x="31.75" y="19.05" smashed="yes" rot="R270">
+<attribute name="NAME" x="31.115" y="18.415" size="1.6764" layer="25" font="vector" ratio="10" rot="R270"/>
+<attribute name="VALUE" x="30.734" y="23.241" size="1.4224" layer="21" font="vector" ratio="10" rot="R270"/>
+</element>
+<element name="R6" library="SPCoast" package="AXIAL-0.4-RES" value="1K" x="26.67" y="19.05" smashed="yes" rot="R270">
+<attribute name="NAME" x="26.035" y="18.415" size="1.6764" layer="25" font="vector" ratio="10" rot="R270"/>
+<attribute name="VALUE" x="25.654" y="21.971" size="1.6764" layer="21" font="vector" ratio="10" rot="R270"/>
 </element>
 <element name="ST1" library="SparkFun-Connectors" package="1X06_LOCK" value="" x="15.24" y="3.81" smashed="yes">
@@
 <attribute name="NAME" x="8.4725" y="1.765" size="0.8128" layer="25" rot="R180"/>
 </element>
+<element name="U$1" library="MRCSLogoBtm" package="MRCSLOGOBTM" value="" x="2.54" y="17.78"/>
+<element name="U$2" library="MRCS-prop65warningBtm" package="CA-PROP65WARNING" value="" x="24.13" y="27.94"/>
 </elements>
 <signals>
@@
 </board>
 </drawing>
+<compatibility>
+<note version="6.3" minversion="6.2.2" severity="warning">
+Since Version 6.2.2 text objects can contain more than one line,
+which will not be processed correctly with this version.
+</note>
+</compatibility>
 </eagle>

Commit message: Updated Documentation and created pdf
documentation
Parts:
- C1: device SparkFun-Capacitors:CAP-PTH-SMALLEZ -> SparkFun-Passives:CAP-PTH-SMALLEZ
Changed lines of the file:
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@@
 <layer number="50" name="dxf" color="7" fill="1" visible="no" active="no"/>
 <layer number="51" name="tDocu" color="7" fill="1" visible="yes" active="yes"/>
-<layer number="52" name="bDocu" color="7" fill="1" visible="yes" active="yes"/>
+<layer number="52" name="bDocu" color="7" fill="1" visible="no" active="yes"/>
 <layer number="53" name="tGND_GNDA" color="7" fill="9" visible="no" active="no"/>
 <layer number="54" name="bGND_GNDA" color="1" fill="9" visible="no" active="no"/>
@@
 <text x="33.02" y="34.29" size="1.016" layer="21" font="vector" ratio="10" rot="R90">M-</text>
 <text x="36.83" y="26.035" size="1.778" layer="52" font="vector" ratio="10" rot="MR270">RSMC V1.9</text>
+<text x="18.415" y="6.985" size="0.8128" layer="125" font="vector">C1</text>
+<text x="8.4725" y="1.76499375" size="0.8128" layer="125" font="vector" rot="R180">CON1</text>
+<text x="5.08" y="32.893" size="0.8128" layer="125" font="vector">J1</text>
+<text x="5.0038" y="34.29" size="0.8128" layer="125" font="vector" ratio="10">J2</text>
+<text x="1.27" y="36.449" size="0.8128" layer="125" font="vector" ratio="10">M1</text>
+<text x="35.56" y="36.449" size="0.8128" layer="125" font="vector" ratio="10">M8</text>
+<text x="36.195" y="7.62" size="1.27" layer="125" font="vector" ratio="10" rot="R270">Q1</text>
+<text x="23.495" y="18.415" size="1.6764" layer="125" font="vector" ratio="10" rot="R270">R3</text>
+<text x="28.575" y="18.415" size="1.6764" layer="125" font="vector" ratio="10" rot="R270">R4</text>
+<text x="31.115" y="18.415" size="1.6764" layer="125" font="vector" ratio="10" rot="R270">R5</text>
+<text x="26.035" y="18.415" size="1.6764" layer="125" font="vector" ratio="10" rot="R270">R6</text>
+<text x="13.97" y="5.588" size="1.27" layer="125" font="vector">ST1</text>
+<text x="12.954" y="19.304" size="0.8128" layer="125" font="vector" ratio="10">U1</text>
 <text x="18.415" y="6.985" size="0.8128" layer="125" font="vector">C1</text>
 <text x="8.4725" y="1.76499375" size="0.8128" layer="125" font="vector" rot="R180">CON1</text>
@@
 </autorouter>
 <elements>
-<element name="C1" library="SparkFun-Capacitors" package="CAP-PTH-SMALLEZ" value=".01uF" x="13.97" y="6.985" smashed="yes">
+<element name="C1" library="SparkFun-Passives" package="CAP-PTH-SMALLEZ" value=".01uF" x="13.97" y="6.985" smashed="yes">
 <attribute name="NAME" x="18.415" y="6.985" size="0.8128" layer="25"/>
 <attribute name="VALUE" x="12.7" y="4.445" size="0.6096" layer="27"/>
